File: Pomodoro_v1.0/Pomodoro_v1.sch (KiCad schematic (older format))
At the start: 74 parts, among them J1 BATT, J10 PE5, J11 PE6, J12 PE7, J13 SWIM, J2 NTC, J3 USB_OTG, J4 LDR, J5 PE0, J6 PE1, J7 PE2, J8 PE3, J9 PE4, Q1 BC807, Q2 BC817, SW1 SLIDER, SW2 BUTTON, U1 MCP73833, U2 TPS62260, U3 STM8L151C2T6

Commit message: add AS1122 to the schematic, started assigning footprints
Parts:
- removed J5: PE0, symbol TEST_1P
- removed J6: PE1, symbol TEST_1P
- removed J7: PE2, symbol TEST_1P
- removed J8: PE3, symbol TEST_1P
- removed Q2: BC817, symbol Q_NPN_BEC
- added C11: 10u, Capacitors_SMD:C_0805, symbol C
- added C12: 100n, Capacitors_SMD:C_0805, symbol C
- added M1, M2, M3, M4: MOUNTING-HOLE, Mounting_Holes:MountingHole_3.2mm_M3_Pad, symbol MOUNTING-HOLE
- added Q2: BC807, TO_SOT_Packages_SMD:SOT-23, symbol BC807
- added R30: 4K7, Resistors_SMD:R_0805, symbol R
- added R31: 0R, Resistors_SMD:R_0805, symbol R
- added TP1: PA3, Measurement_Points:Measurement_Point_Round-SMD-Pad_Small, symbol TEST_1P
- added TP13: PF0, Measurement_Points:Measurement_Point_Round-SMD-Pad_Small, symbol TEST_1P
- added TP2: PA4, Measurement_Points:Measurement_Point_Round-SMD-Pad_Small, symbol TEST_1P
- added TP3: PA7, Measurement_Points:Measurement_Point_Round-SMD-Pad_Small, symbol TEST_1P
- added TP4: PC0, Measurement_Points:Measurement_Point_Round-SMD-Pad_Small, symbol TEST_1P
- added TP5: PC1, Measurement_Points:Measurement_Point_Round-SMD-Pad_Small, symbol TEST_1P
- added TP6: PC6, Measurement_Points:Measurement_Point_Round-SMD-Pad_Small, symbol TEST_1P
- added TP7: PC7, Measurement_Points:Measurement_Point_Round-SMD-Pad_Small, symbol TEST_1P
- added TP8: PD7, Measurement_Points:Measurement_Point_Round-SMD-Pad_Small, symbol TEST_1P
- added U4: AS1122, symbol AS1122
- C1, C10, C2, C3, C4, C5, C6, C7, C8, C9: footprint (none) -> Capacitors_SMD:C_0805
- D1, D10, D2, D3, D4, D5, D6, D7, D8, D9: footprint (none) -> LEDs:LED_0805
- J1, J2: footprint (none) -> Connectors_JST:JST_PH_S2B-PH-K_02x2.00mm_Angled
- J13: footprint (none) -> Connectors_JST:JST_PH_B4B-PH-K_04x2.00mm_Straight
- J3: footprint (none) -> Connectors_USB:USB_Micro-B_Molex-105017-0001
- J4: footprint (none) -> Pin_Headers:Pin_Header_Straight_1x02_Pitch2.54mm
- J5: renamed from J?; footprint (none) -> Pin_Headers:Pin_Header_Straight_1x03_Pitch2.54mm
- L2: footprint (none) -> Inductors_SMD:L_0805
- R1, R10, R11, R12, R13, R14, R15, R16, R17, R18, R19, R2, R20, R21, R22, R23, R24, R25, R28, R29, R3, R4, R5, R6, R7, R8, R9: footprint (none) -> Resistors_SMD:R_0805
- R26: value R -> 10K; footprint (none) -> Resistors_SMD:R_0805
- R27: value R -> 16K2; footprint (none) -> Resistors_SMD:R_0805
- TP10: renamed from J10; footprint (none) -> Measurement_Points:Measurement_Point_Round-SMD-Pad_Small
- TP11: renamed from J11; footprint (none) -> Measurement_Points:Measurement_Point_Round-SMD-Pad_Small
- TP12: renamed from J12; footprint (none) -> Measurement_Points:Measurement_Point_Round-SMD-Pad_Small
- TP9: renamed from J9; footprint (none) -> Measurement_Points:Measurement_Point_Round-SMD-Pad_Small
- U1: footprint (none) -> Housings_DFN_QFN:DFN-10-1EP_3x3mm_Pitch0.5mm
Connections:
- net labels added: AS_CLK, AS_IRQ, AS_RST, AS_SD, D0_0, D0_1, D0_10, D0_11, D0_2, D0_3, D0_4, D0_5, D0_6, D0_7, D0_8, D0_9, DO_1, DO_10, DO_11, DO_2, DO_3, DO_4, DO_5, DO_6, DO_7, DO_8, DO_9
- wire segments 203 -> 258
- no-connect marks 6 -> 7
Other:
- note added: "8mA"
- note added: "MOUNTING\nHOLES"

Commit message: latop update
Parts:
- removed J4: LDR, Pin_Headers:Pin_Header_Straight_1x02_Pitch2.54mm, symbol Conn_01x02
- added R32: R_PHOTO, symbol R_PHOTO
- BZ1: footprint (none) -> BUZZERS_TDK:BUZZERS_TDK
- D1, D2: Link (none) -> https://www.tme.eu/pl/details/osr50805c1e/diody-led-smd-kol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
- D10, D7, D8, D9: Link (none) -> https://www.tme.eu/pl/details/ll-s170pgc-g5-1a/diody-led-sm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
- D11: footprint (none) -> LEDs:LED_RGB_5050-6; Link (none) -> https://www.tme.eu/pl/details/fyls-5050nrgbc/diody-led-smd-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
- D3, D4, D5, D6: Link (none) -> https://www.tme.eu/pl/details/osy50805c1e/diody-led-smd-kol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
- J3: Link (none) -> https://www.tme.eu/pl/details/mx-105017-0001/zlacza-usb-i-i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
- L1: footprint (none) -> LPS3015:LPS3015
- Q1, Q2: Link (none) -> https://pl.mouser.com/ProductDetail/Nexperia/BC807215?qs=sG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
- R1, R2: value R -> 200R; Link (none) -> https://www.tme.eu/pl/details/smd0805-200r/rezystory-smd-08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
- R11, R12, R13, R14: value R -> 10R; Link (none) -> https://www.tme.eu/pl/details/smd0805-10r/rezystory-smd-080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
- R15, R16: value R -> 0R
- R17, R3, R4, R6, R9: value R -> 200R
- SW1: Link (none) -> https://www.tme.eu/pl/details/5ms1s102am6qe/przelaczniki-su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
- SW2: Link (none) -> https://www.tme.eu/pl/details/tacts-24n-f/mikroprzelaczniki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
- U1: Link (none) -> https://www.tme.eu/pl/details/mcp73833-fci_mf/kontrolery-ba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
- U2: footprint (none) -> TO_SOT_Packages_SMD:SOT-23-5; Link (none) -> https://pl.mouser.com/ProductDetail/Texas-Instruments/TPS62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
- U3: footprint (none) -> Housings_QFP:LQFP-48_7x7mm_Pitch0.5mm; Link (none) -> https://pl.mouser.com/ProductDetail/STMicroelectronics/STM8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
- U3: footprint (none) -> Housings_QFP:LQFP-48_7x7mm_Pitch0.5mm
- U4: footprint (none) -> Housings_DFN_QFN:QFN-24_4x4mm_Pitch0.5mm; Link (none) -> https://pl.mouser.com/ProductDetail/STMicroelectronics/STM8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
- U4: footprint (none) -> Housings_DFN_QFN:QFN-24_4x4mm_Pitch0.5mm; Link (none) -> https://pl.mouser.com/ProductDetail/ams/AS1122-BQFT?qs=sGAE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
Connections:
- wire segments 258 -> 257
Other:
- note added: "LED\nDRIVER"

Commit message: assign footprints
Parts:
- removed SW2: BUTTON, symbol SW_Push_Dual
- added SW2: BUTTON_SPST, NINIGI TACTS-24N-F:NINIGI TACTS-24N-F, symbol BUTTON_SPST
- R18: value R -> 66k5; Link (none) -> https://www.tme.eu/pl/details/crcw080566k5fktabc/rezystory-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
- R20: value R -> 1k6; Link (none) -> https://www.tme.eu/pl/details/crcw08051k60fktabc/rezystory-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
- R32: footprint (none) -> Pin_Headers:Pin_Header_Straight_1x02_Pitch2.54mm
- SW1: footprint (none) -> SLIDE_SWITCHES: 5MS1S102AM6QE
- U4: footprint Housings_DFN_QFN:QFN-24_4x4mm_Pitch0.5mm -> Housings_DFN_QFN:QFN-24_4x4mm_Pitch0.5mm_NoMask
