File: Pomodoro_v1.0/Pomodoro_v1.sch (KiCad schematic (older format))
At the start: 88 parts, among them J1 BATT, J13 SWIM, J2 NTC, J3 USB_OTG, J5 UART, M1 MOUNTING-HOLE, M2 MOUNTING-HOLE, M3 MOUNTING-HOLE, M4 MOUNTING-HOLE, Q1 BC807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

Commit message: Components placement done, initial routing (power tracks)
Parts:
- removed J1: BATT, Connectors_JST:JST_PH_S2B-PH-K_02x2.00mm_Angled, symbol Conn_01x02
- removed J2: NTC, Connectors_JST:JST_PH_S2B-PH-K_02x2.00mm_Angled, symbol Conn_01x02
- added C13, C14: 10u, Capacitors_SMD:C_0805, symbol C
- added J1: BATT, Connectors_JST:s3b-ph-kl, symbol Conn_01x03
- added R33: 0R, Resistors_SMD:R_0805, symbol R
- added R34: 10K, Resistors_SMD:R_0805, symbol R
Connections:
- wire segments 257 -> 312

Commit message: fix STAT_x/STATx typo
Connections:
- net labels removed: STAT_1, STAT_2
- wire segments 312 -> 258
Changed lines of the file:
@@
 LIBS:MCU_ST_STM8
 LIBS:button_spst
-LIBS:Pomodoro_v1-cache
 EELAYER 25 0
 EELAYER END
@@
 $EndComp
 Text Label 8050 3550 0    60   ~ 0
-STAT_1
+STAT1
 Text Label 8050 3650 0    60   ~ 0
-STAT_2
+STAT2
 $Comp
 L VCC #PWR035
@@
 	4100 2800 4050 2800
 Wire Wire Line
-	4100 2650 4100 2700
-Wire Wire Line
-	4100 2700 4100 2800
+	4100 2650 4100 2800
 Wire Wire Line
 	4050 2700 4100 2700
@@
 	3000 2800 3050 2800
 Wire Wire Line
-	3000 2650 3000 2700
-Wire Wire Line
-	3000 2700 3000 2800
+	3000 2650 3000 2800
 Wire Wire Line
 	3050 2700 3000 2700
@@
 	1200 1700 1200 1650
 Wire Wire Line
-	2400 700  2400 750
-Wire Wire Line
-	2400 750  2400 800
+	2400 700  2400 800
 Wire Wire Line
 	2100 1000 1950 1000
 Wire Wire Line
-	1950 750  1950 1000
-Wire Wire Line
-	1950 1000 1950 1050
-Wire Wire Line
-	2400 1200 2400 1250
-Wire Wire Line
-	2400 1250 2400 1400
-Wire Wire Line
-	4050 3000 4300 3000
-Wire Wire Line
-	4300 3000 4900 3000
-Wire Wire Line
-	4050 2900 4500 2900
-Wire Wire Line
-	4500 2900 4900 2900
+	1950 750  1950 1050
+Wire Wire Line
+	2400 1200 2400 1400
+Wire Wire Line
+	4050 3000 4900 3000
+Wire Wire Line
+	4050 2900 4900 2900
 Wire Wire Line
 	1950 1500 1650 1500
@@
 	650  4700 650  4750
 Wire Wire Line
-	650  4750 700  4750
-Wire Wire Line
-	700  4750 750  4750
+	650  4750 750  4750
 Wire Wire Line
 	750  4750 750  4700
@@
 	3050 3000 2800 3000
 Wire Wire Line
-	800  2700 1050 2700
-Wire Wire Line
-	1050 2700 1100 2700
+	800  2700 1100 2700
 Wire Wire Line
 	1050 2750 1050 2700
@@
 	3800 1050 3850 1050
 Wire Wire Line
-	4100 1400 4100 1450
-Wire Wire Line
-	4100 1450 4100 1500
+	4100 1400 4100 1500
 Wire Wire Line
 	3800 1250 4000 1250
@@
 	4000 1250 4000 1450
 Wire Wire Line
-	4000 1450 4100 1450
-Wire Wire Line
-	4100 1450 4350 1450
+	4000 1450 4350 1450
 Connection ~ 4100 1450
 Wire Wire Line
-	4050 1050 4100 1050
-Wire Wire Line
-	4100 1050 4350 1050
-Wire Wire Line
-	4350 1050 4700 1050
-Wire Wire Line
-	4700 1000 4700 1050
-Wire Wire Line
-	4700 1050 4700 1100
+	4050 1050 4700 1050
+Wire Wire Line
+	4700 1000 4700 1100
 Wire Wire Line
 	4350 1100 4350 1050
@@
 	8800 1950 7950 1950
 Wire Wire Line
-	6800 3350 6800 3400
-Wire Wire Line
-	6800 3400 6800 3450
-Wire Wire Line
-	6600 3400 6800 3400
-Wire Wire Line
-	6800 3400 7300 3400
+	6800 3350 6800 3450
+Wire Wire Line
+	6600 3400 7300 3400
 Connection ~ 6800 3400
 Wire Wire Line
-	6800 3750 6800 3800
-Wire Wire Line
-	6800 3800 6800 3850
+	6800 3750 6800 3850
 Wire Wire Line
 	6800 3000 6800 3050
@@
 	5850 7300 5800 7300
 Wire Wire Line
-	5800 7300 5800 7400
-Wire Wire Line
-	5800 7400 5800 7450
+	5800 7300 5800 7450
 Wire Wire Line
 	5850 7400 5800 7400
@@
 	5850 7050 5800 7050
 Wire Wire Line
-	5800 7050 5800 6900
-Wire Wire Line
-	5400 6900 5450 6900
-Wire Wire Line
-	5450 6900 5650 6900
-Wire Wire Line
-	5650 6900 5800 6900
-Wire Wire Line
-	5800 6900 5850 6900
+	5800 6900 5800 7050
+Wire Wire Line
+	5400 6900 5850 6900
 Connection ~ 5800 6900
 Wire Wire Line
 	5650 7300 5650 7250
 Wire Wire Line
-	5450 7300 5550 7300
-Wire Wire Line
-	5550 7300 5650 7300
+	5450 7300 5650 7300
 Wire Wire Line
 	5450 7300 5450 7250
@@
 	5800 6800 5850 6800
 Wire Wire Line
-	5800 6650 5800 6700
-Wire Wire Line
-	5800 6700 5800 6800
+	5800 6650 5800 6800
 Wire Wire Line
 	5850 6700 5800 6700
 Connection ~ 5800 6700
 Wire Wire Line
-	5750 6150 6000 6150
-Wire Wire Line
-	6000 6150 6250 6150
+	5750 6150 6250 6150
 Wire Wire Line
 	5750 6150 5750 6100
 Wire Wire Line
-	6000 6100 6000 6150
-Wire Wire Line
-	6000 6150 6000 6200
+	6000 6100 6000 6200
 Connection ~ 6000 6150
 Wire Wire Line
-	5750 5750 6000 5750
-Wire Wire Line
-	6000 5750 6250 5750
+	5750 5750 6250 5750
 Wire Wire Line
 	5750 5750 5750 5800
 Wire Wire Line
-	6000 5700 6000 5750
-Wire Wire Line
-	6000 5750 6000 5800
+	6000 5700 6000 5800
 Connection ~ 6000 5750
 Wire Wire Line
@@
 	8200 1200 8200 1250
 Wire Wire Line
-	6400 2100 6400 2200
-Wire Wire Line
-	6400 2200 6400 2250
+	6400 2100 6400 2250
 Wire Wire Line
 	6400 2100 6350 2100
@@
 	5650 2200 5600 2200
 Wire Wire Line
-	5600 2200 5600 2100
-Wire Wire Line
-	5150 2100 5550 2100
-Wire Wire Line
-	5550 2100 5600 2100
-Wire Wire Line
-	5600 2100 5650 2100
+	5600 2100 5600 2200
+Wire Wire Line
+	5150 2100 5650 2100
 Wire Wire Line
 	5550 2050 5550 2100
@@
 	4300 2500 4300 2450
 Wire Wire Line
-	4300 2450 4400 2450
-Wire Wire Line
-	4400 2450 4500 2450
+	4300 2450 4500 2450
 Wire Wire Line
 	4500 2450 4500 2500
@@
 	8350 3650 8050 3650
 Wire Wire Line
-	5600 2950 5600 3000
-Wire Wire Line
-	5600 3000 5600 3200
-Wire Wire Line
-	5100 3400 5500 3400
-Wire Wire Line
-	5500 3400 5600 3400
+	5600 2950 5600 3200
+Wire Wire Line
+	5100 3400 5600 3400
 Wire Wire Line
 	5500 3400 5500 3350
@@
 	5150 3700 5150 3800
 Wire Wire Line
-	5150 3800 5300 3800
-Wire Wire Line
-	5300 3800 5400 3800
-Wire Wire Line
-	5400 3800 5500 3800
-Wire Wire Line
-	5500 3800 5650 3800
+	5150 3800 5650 3800
 Wire Wire Line
 	5650 3800 5650 3700
@@
 	800  5800 800  5750
 Wire Wire Line
-	800  5750 1050 5750
-Wire Wire Line
-	1050 5750 1400 5750
-Wire Wire Line
-	1400 5750 1650 5750
-Wire Wire Line
-	1650 5750 1900 5750
-Wire Wire Line
-	1900 5750 2050 5750
-Wire Wire Line
-	2050 5750 2150 5750
-Wire Wire Line
-	2150 5750 2500 5750
-Wire Wire Line
-	2500 5750 2750 5750
-Wire Wire Line
-	2750 5750 3000 5750
-Wire Wire Line
-	3000 5750 3250 5750
-Wire Wire Line
-	3250 5750 3700 5750
-Wire Wire Line
-	3700 5750 3900 5750
-Wire Wire Line
-	3900 5750 4100 5750
+	800  5750 4100 5750
 Wire Wire Line
 	3250 5750 3250 5800
@@
 	4150 4800 4100 4800
 Wire Wire Line
-	4100 4700 4100 4800
-Wire Wire Line
-	4100 4800 4100 4850
+	4100 4700 4100 4850
 Wire Wire Line
 	4150 4700 4100 4700
@@
 	3350 3800 3350 3750
 Wire Wire Line
-	3350 3750 3500 3750
-Wire Wire Line
-	3500 3750 3650 3750
+	3350 3750 3650 3750
 Wire Wire Line
 	3650 3750 3650 3800
@@
 	3350 4100 3350 4150
 Wire Wire Line
-	3350 4150 3500 4150
-Wire Wire Line
-	3500 4150 3650 4150
+	3350 4150 3650 4150
 Wire Wire Line
 	3650 4150 3650 4100
@@
 $EndComp
 Wire Wire Line
-	7000 2000 7000 2050
-Wire Wire Line
-	7000 2050 7000 2100
+	7000 2000 7000 2100
 Wire Wire Line
 	7000 2400 7000 2450
@@
 	2950 1050 3000 1050
 Wire Wire Line
-	2950 1050 2950 850
-Wire Wire Line
-	2950 850  2950 800
+	2950 800  2950 1050
 Wire Wire Line
 	2850 900  2850 850
@@
 	2850 1200 2850 1250
 Wire Wire Line
-	2850 1250 3000 1250
-Wire Wire Line
-	2400 1250 2850 1250
-$Comp
-L +4V #PWR?
+	2400 1250 3000 1250
+$Comp
+L +4V #PWR048
 U 1 1 5B781BAA
 P 1600 700
-F 0 "#PWR?" H 1600 550 50  0001 C CNN
+F 0 "#PWR048" H 1600 550 50  0001 C CNN
 F 1 "+4V" H 1600 840 50  0000 C CNN
 F 2 "" H 1600 700 50  0001 C CNN

Commit message: fix D0_x -> DO_x typo
Parts:
- U4: symbol AS1122 -> AS1122-RESCUE-Pomodoro_v1
Connections:
- net labels added: DO_0
- net labels removed: D0_0, D0_1, D0_10, D0_11, D0_2, D0_3, D0_4, D0_5, D0_6, D0_7, D0_8, D0_9
Changed lines of the file:
@@
 EESchema Schematic File Version 2
+LIBS:Pomodoro_v1-rescue
 LIBS:power
 LIBS:device
@@
 LIBS:MCU_ST_STM8
 LIBS:button_spst
+LIBS:Pomodoro_v1-cache
 EELAYER 25 0
 EELAYER END
@@
 MOUNTING\nHOLES
 $Comp
-L AS1122 U4
+L AS1122-RESCUE-Pomodoro_v1 U4
 U 1 1 5B2F9CCE
 P 2400 3600
@@
 $EndComp
 $Comp
-L AS1122 U4
+L AS1122-RESCUE-Pomodoro_v1 U4
 U 2 1 5B2F9DE7
 P 4350 4150
@@
 	5850 7050 5800 7050
 Wire Wire Line
-	5800 6900 5800 7050
+	5800 7050 5800 6900
 Wire Wire Line
 	5400 6900 5850 6900
@@
 	5650 2200 5600 2200
 Wire Wire Line
-	5600 2100 5600 2200
+	5600 2200 5600 2100
 Wire Wire Line
 	5150 2100 5650 2100
@@
 	800  6100 800  6400
 Text Label 800  6350 1    60   ~ 0
-D0_0
+DO_0
 Text Label 1050 6350 1    60   ~ 0
 DO_1
@@
 	2900 3700 3100 3700
 Text Label 3100 3700 2    60   ~ 0
-D0_0
+DO_0
 Wire Wire Line
 	2900 3800 3100 3800
@@
 	2900 4800 3150 4800
 Text Label 3100 3800 2    60   ~ 0
-D0_1
+DO_1
 Text Label 3100 3900 2    60   ~ 0
-D0_2
+DO_2
 Text Label 3100 4000 2    60   ~ 0
-D0_3
+DO_3
 Text Label 3100 4100 2    60   ~ 0
-D0_4
+DO_4
 Text Label 3100 4200 2    60   ~ 0
-D0_5
+DO_5
 Text Label 3100 4300 2    60   ~ 0
-D0_6
+DO_6
 Text Label 3100 4400 2    60   ~ 0
-D0_7
+DO_7
 Text Label 3100 4500 2    60   ~ 0
-D0_8
+DO_8
 Text Label 3100 4600 2    60   ~ 0
-D0_9
+DO_9
 Text Label 3150 4700 2    60   ~ 0
-D0_10
+DO_10
 Text Label 3150 4800 2    60   ~ 0
-D0_11
+DO_11
 Wire Wire Line
 	3800 4250 4150 4250
